Commit message: 拆分模型文件

File: src/robot_description/urdf/humanoid.urdf.xacro (robot description, xacro)
@@ -1,1507 +1,11 @@
-<?xml version="1.0" encoding="utf-8"?>
-<robot
-  name="humanoid" xmlns:xacro="http://www.ros.org/wiki/xacro">
-  <link
-    name="base_link">
-    <inertial>
-      <origin
-        xyz="1.07784451355147E-06 0.0284280497758001 0.0930501056429116"
-        rpy="0 0 0" />
-      <mass
-        value="25.2827775843096" />
-      <inertia
-        ixx="1.05306308303982"
-        ixy="5.35850857338871E-07"
-        ixz="-8.40544864225828E-06"
-        iyy="0.379347819173407"
-        iyz="4.4668154477851E-06"
-        izz="1.39119566760917" />
-    </inertial>
-    <visual>
-      <origin
-        xyz="0 0 0"
-        rpy="0 0 0" />
-      <geometry>
-        <mesh
-          filename="package://robot_description/meshes/base_link.STL" />
-      </geometry>
-      <material
-        name="">
-        <color
-          rgba="0.792156862745098 0.819607843137255 0.929411764705882 1" />
-      </material>
-    </visual>
-    <collision>
-      <origin
-        xyz="0 0 0"
-        rpy="0 0 0" />
-      <geometry>
-        <mesh
-          filename="package://robot_description/meshes/base_link.STL" />
-      </geometry>
-    </collision>
-  </link>
-  <link
-    name="neck_pitch_link">
-    <inertial>
-      <origin
-        xyz="7.01840304657472E-05 0.130777470021731 -0.00331694653990108"
-        rpy="0 0 0" />
-      <mass
-        value="0.148218827310183" />
-      <inertia
-        ixx="9.52279837773781E-05"
-        ixy="-9.91190135430179E-08"
-        ixz="1.98844059206848E-07"
-        iyy="7.30070921223501E-05"
-        iyz="3.47609457314995E-06"
-        izz="9.0131560532935E-05" />
-    </inertial>
-    <visual>
-      <origin
-        xyz="0 0 0"
-        rpy="0 0 0" />
-      <geometry>
-        <mesh
-          filename="package://robot_description/meshes/neck_pitch_link.STL" />
-      </geometry>
-      <material
-        name="">
-        <color
-          rgba="0.647058823529412 0.619607843137255 0.588235294117647 1" />
-      </material>
-    </visual>
-    <collision>
-      <origin
-        xyz="0 0 0"
-        rpy="0 0 0" />
-      <geometry>
-        <mesh
-          filename="package://robot_description/meshes/neck_pitch_link.STL" />
-      </geometry>
-    </collision>
-  </link>
-  <joint
-    name="neck_pitch_joint"
-    type="revolute">
-    <origin
-      xyz="0 0.189998253900838 0.835499049600994"
-      rpy="1.5707963267949 0 1.5707963267949" />
-    <parent
-      link="base_link" />
-    <child
-      link="neck_pitch_link" />
-    <axis
-      xyz="0 1 0" />
-    <limit
-      lower="-3.14"
-      upper="3.14"
-      effort="20.0"
-      velocity="50.0" />
-  </joint>
-  <link
-    name="neck_yaw_link">
-    <inertial>
-      <origin
-        xyz="-0.00016459752079714 0.00712784323803106 -0.0394648436747978"
-        rpy="0 0 0" />
-      <mass
-        value="0.0765456211575113" />
-      <inertia
-        ixx="3.23897327523942E-05"
-        ixy="-2.65902764441305E-14"
-        ixz="-5.98960713926039E-15"
-        iyy="1.63880392625728E-05"
-        iyz="5.16658827031463E-07"
-        izz="4.47591140398881E-05" />
-    </inertial>
-    <visual>
-      <origin
-        xyz="0 0 0"
-        rpy="0 0 0" />
-      <geometry>
-        <mesh
-          filename="package://robot_description/meshes/neck_yaw_link.STL" />
-      </geometry>
-      <material
-        name="">
-        <color
-          rgba="1 1 1 0.25" />
-      </material>
-    </visual>
-    <collision>
-      <origin
-        xyz="0 0 0"
-        rpy="0 0 0" />
-      <geometry>
-        <mesh
-          filename="package://robot_description/meshes/neck_yaw_link.STL" />
-      </geometry>
-    </collision>
-  </link>
-  <joint
-    name="neck_yaw_joint"
-    type="revolute">
-    <origin
-      xyz="0.000164597494633156 0.135935192091684 0.0268002104136432"
-      rpy="0 0 0" />
-    <parent
-      link="neck_pitch_link" />
-    <child
-      link="neck_yaw_link" />
-    <axis
-      xyz="0 0 1" />
-    <limit
-      lower="-3.14"
-      upper="3.14"
-      effort="20.0"
-      velocity="50.0" />
-  </joint>
-  <link
-    name="head_link">
-    <inertial>
-      <origin
-        xyz="-0.0538137633177245 4.16333634234434E-17 0"
-        rpy="0 0 0" />
-      <mass
-        value="0.398240212565594" />
-      <inertia
-        ixx="0.00225801965865169"
-        ixy="3.25260651745651E-19"
-        ixz="2.29715335295366E-18"
-        iyy="0.00143841223628256"
-        iyz="-1.12485975395371E-18"
-        izz="0.00239435389760271" />
-    </inertial>
-    <visual>
-      <origin
-        xyz="0 0 0"
-        rpy="0 0 0" />
-      <geometry>
-        <mesh
-          filename="package://robot_description/meshes/head_link.STL" />
-      </geometry>
-      <material
-        name="">
-        <color
-          rgba="1 1 1 1" />
-      </material>
-    </visual>
-    <collision>
-      <origin
-        xyz="0 0 0"
-        rpy="0 0 0" />
-      <geometry>
-        <mesh
-          filename="package://robot_description/meshes/head_link.STL" />
-      </geometry>
-    </collision>
-  </link>
-  <joint
-    name="head_neck_joint"
-    type="fixed">
-    <origin
-      xyz="0.0498354025053677 0.109164807908296 -0.0267999999999801"
-      rpy="-1.5707963267949 0 0" />
-    <parent
-      link="neck_yaw_link" />
-    <child
-      link="head_link" />
-    <axis
-      xyz="0 0 0" />
-    <limit
-      lower="3.14"
-      upper="3.14"
-      effort="3.14"
-      velocity="3.14" />
-  </joint>
-  <link name="head_camera_link">
-    <collision>
-      <geometry>
-        <box size="0.0001 0.0001 0.0001"/>
-      </geometry>
-    </collision>
-  </link>
-  <joint
-    name="head_camera_joint"
-    type="fixed">
-    <parent link="head_link"/>
-    <child link="head_camera_link"/>
-    <origin xyz="0 0 0" rpy="-1.57079632679 0 -1.57079632679"/>
-  </joint>
-  <!-- 右臂 -->
-  <link
-    name="right_base_pitch_link">
-    <inertial>
-      <origin
-        xyz="-0.0394540906091678 -0.00117049156839028 0.0362772096702395"
-        rpy="0 0 0" />
-      <mass
-        value="0.244817289982652" />
-      <inertia
-        ixx="0.00042258611468929"
-        ixy="-3.33213778042763E-07"
-        ixz="6.13148868322963E-05"
-        iyy="0.00043362815715413"
-        iyz="1.84861840406614E-06"
-        izz="0.000449580199614448" />
-    </inertial>
-    <visual>
-      <origin
-        xyz="0 0 0"
-        rpy="0 0 0" />
-      <geometry>
-        <mesh
-          filename="package://robot_description/meshes/right_base_pitch_link.STL" />
-      </geometry>
-      <material
-        name="">
-        <color
-          rgba="1 1 1 1" />
-      </material>
-    </visual>
-    <collision>
-      <origin
-        xyz="0 0 0"
-        rpy="0 0 0" />
-      <geometry>
-        <mesh
-          filename="package://robot_description/meshes/right_base_pitch_link.STL" />
-      </geometry>
-    </collision>
-  </link>
-  <joint
-    name="right_base_pitch_joint"
-    type="revolute">
-    <origin
-      xyz="0.21400441954841 0.189998253900819 0.822999049601032"
-      rpy="1.5707963267949 0 1.5707963267949" />
-    <parent
-      link="base_link" />
-    <child
-      link="right_base_pitch_link" />
-    <axis
-      xyz="0 0 -1" />
-    <limit
-      lower="-3.14"
-      upper="3.14"
-      effort="20.0"
-      velocity="50.0" />
-  </joint>
-  <link
-    name="right_shoulder_roll_link">
-    <inertial>
-      <origin
-        xyz="-0.0504751969032359 -2.3505993093087E-06 -0.0382593125478601"
-        rpy="0 0 0" />
-      <mass
-        value="0.219562602027133" />
-      <inertia
-        ixx="0.000414250305228579"
-        ixy="-5.1544201930132E-09"
-        ixz="-8.79018796006794E-05"
-        iyy="0.000412104091228023"
-        iyz="-6.24422590434745E-08"
-        izz="0.000365288665382115" />
-    </inertial>
-    <visual>
-      <origin
-        xyz="0 0 0"
-        rpy="0 0 0" />
-      <geometry>
-        <mesh
-          filename="package://robot_description/meshes/right_shoulder_roll_link.STL" />
-      </geometry>
-      <material
-        name="">
-        <color
-          rgba="1 1 1 1" />
-      </material>
-    </visual>
-    <collision>
-      <origin
-        xyz="0 0 0"
-        rpy="0 0 0" />
-      <geometry>
-        <mesh
-          filename="package://robot_description/meshes/right_shoulder_roll_link.STL" />
-      </geometry>
-    </collision>
-  </link>
-  <joint
-    name="right_shoulder_roll_joint"
-    type="revolute">
-    <origin
-      xyz="0.0512767086241353 0.00154568843845215 0.070000086877735"
-      rpy="1.57079632679489 -0.0124370994640314 1.60093654227117" />
-    <parent
-      link="right_base_pitch_link" />
-    <child
-      link="right_shoulder_roll_link" />
-    <axis
-      xyz="0 0 -1" />
-    <limit
-      lower="-3.14"
-      upper="3.14"
-      effort="20.0"
-      velocity="50.0" />
-  </joint>
-  <link
-    name="right_shoulder_yaw_link">
-    <inertial>
-      <origin
-        xyz="-0.020385273211367 -8.15235141520682E-06 0.0357353445479509"
-        rpy="0 0 0" />
-      <mass
-        value="0.106143604615312" />
-      <inertia
-        ixx="9.66386839936161E-05"
-        ixy="-4.74531869270227E-09"
-        ixz="2.12882628388833E-05"
-        iyy="0.000122064598284769"
-        iyz="-6.1579299009481E-08"
-        izz="0.00010313012003071" />
-    </inertial>
-    <visual>
-      <origin
-        xyz="0 0 0"
-        rpy="0 0 0" />
-      <geometry>
-        <mesh
-          filename="package://robot_description/meshes/right_shoulder_yaw_link.STL" />
-      </geometry>
-      <material
-        name="">
-        <color
-          rgba="1 1 1 1" />
-      </material>
-    </visual>
-    <collision>
-      <origin
-        xyz="0 0 0"
-        rpy="0 0 0" />
-      <geometry>
-        <mesh
-          filename="package://robot_description/meshes/right_shoulder_yaw_link.STL" />
-      </geometry>
-    </collision>
-  </link>
-  <joint
-    name="right_shoulder_yaw_joint"
-    type="revolute">
-    <origin
-      xyz="-0.161499730454391 0 -0.0674997882054564"
-      rpy="1.5707963267949 -0.209915812016821 -1.5707963267949" />
-    <parent
-      link="right_shoulder_roll_link" />
-    <child
-      link="right_shoulder_yaw_link" />
-    <axis
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
Commit message: 命名修改、urdf结构调整

File: src/robot_description/urdf/humanoid.urdf.xacro (robot description, xacro)
@@ -4,4 +4,7 @@
   <!-- 包含结构 -->
   <xacro:include filename="robot_structure.urdf.xacro"/>
+  <!-- 包含 相机光学坐标系 -->
+  <xacro:include filename="camera_optical_link.xacro"/>
+  <xacro:camera_optical_link/>
   <xacro:if value="$(arg use_gazebo)">
     <!-- gazebo 仿真 -->

File: src/robot_description/urdf/robot_gazebo.xacro (robot description, xacro)
@@ -30,5 +30,5 @@
     </gazebo>
     <!-- 右手相机（RGB） -->
-    <gazebo reference="right_camera_link">
+    <gazebo reference="left_camera_optical_link">
       <sensor name="right_camera" type="camera">
         <pose>0 0 0 0 -1.5708 1.5708</pose>
@@ -51,5 +51,5 @@
     </gazebo>
     <!-- 左手相机（RGB） -->
-    <gazebo reference="left_camera_link">
+    <gazebo reference="left_camera_optical_link">
       <sensor name="left_camera" type="camera">
         <pose>0 0 0 1.5708 -1.5708 0</pose>

File: src/robot_description/urdf/robot_structure.urdf.xacro (robot description, xacro)
@@ -697,5 +697,5 @@
   </joint>
   <link
-    name="right_camera_bracket_link">
+    name="right_camera_link">
     <inertial>
       <origin
@@ -718,24 +718,24 @@
       <geometry>
         <mesh
-          filename="package://robot_description/meshes/right_camera_bracket_link.STL" />
-      </geometry>
-      <material
-        name="">
-        <color
-          rgba="1 1 1 1" />
-      </material>
-    </visual>
-    <collision>
-      <origin
-        xyz="0 0 0"
-        rpy="0 0 0" />
-      <geometry>
-        <mesh
-          filename="package://robot_description/meshes/right_camera_bracket_link.STL" />
-      </geometry>
-    </collision>
-  </link>
-  <joint
-    name="right_camera_bracket_joint"
+          filename="package://robot_description/meshes/right_camera_link.STL" />
+      </geometry>
+      <material
+        name="">
+        <color
+          rgba="1 1 1 1" />
+      </material>
+    </visual>
+    <collision>
+      <origin
+        xyz="0 0 0"
+        rpy="0 0 0" />
+      <geometry>
+        <mesh
+          filename="package://robot_description/meshes/right_camera_link.STL" />
+      </geometry>
+    </collision>
+  </link>
+  <joint
+    name="right_camera_joint"
     type="fixed">
     <origin
@@ -745,5 +745,5 @@
       link="right_wrist_yaw_link" />
     <child
-      link="right_camera_bracket_link" />
+      link="right_camera_link" />
     <axis
       xyz="0.0790644615829094 0.996083645985627 0.0395750061855195" />
@@ -753,18 +753,4 @@
       effort="3.14"
       velocity="3.14" />
-  </joint>
-  <link name="right_camera_link">
-    <collision>
-      <geometry>
-        <box size="0.0001 0.0001 0.0001"/>
-      </geometry>
-    </collision>
-  </link>
-  <joint
-    name="right_camera_joint"
-    type="fixed">
-    <parent link="right_camera_bracket_link"/>
-    <child link="right_camera_link"/>
-    <origin xyz="0 0 0" rpy="0 1.57079632679 0"/>
   </joint>
   <!-- 左臂 -->
@@ -1235,5 +1221,5 @@
   </joint>
   <link
-    name="left_camera_bracket_link">
+    name="left_camera_link">
     <inertial>
       <origin
@@ -1256,24 +1242,24 @@
       <geometry>
         <mesh
-          filename="package://robot_description/meshes/left_camera_bracket_link.STL" />
-      </geometry>
-      <material
-        name="">
-        <color
-          rgba="1 1 1 1" />
-      </material>
-    </visual>
-    <collision>
-      <origin
-        xyz="0 0 0"
-        rpy="0 0 0" />
-      <geometry>
-        <mesh
-          filename="package://robot_description/meshes/left_camera_bracket_link.STL" />
-      </geometry>
-    </collision>
-  </link>
-  <joint
-    name="left_camera_bracket_joint"
+          filename="package://robot_description/meshes/left_camera_link.STL" />
+      </geometry>
+      <material
+        name="">
+        <color
+          rgba="1 1 1 1" />
+      </material>
+    </visual>
+    <collision>
+      <origin
+        xyz="0 0 0"
+        rpy="0 0 0" />
+      <geometry>
+        <mesh
+          filename="package://robot_description/meshes/left_camera_link.STL" />
+      </geometry>
+    </collision>
+  </link>
+  <joint
+    name="left_camera_joint"
     type="fixed">
     <origin
@@ -1283,5 +1269,5 @@
       link="left_wrist_yaw_link" />
     <child
-      link="left_camera_bracket_link" />
+      link="left_camera_link" />
     <axis
       xyz="0 0 0" />
@@ -1292,17 +1278,3 @@
       velocity="3.14" />
   </joint>
-  <link name="left_camera_link">
-    <collision>
-      <geometry>
-        <box size="0.0001 0.0001 0.0001"/>
-      </geometry>
-    </collision>
-  </link>
-  <joint
-    name="left_camera_joint"
-    type="fixed">
-    <parent link="left_camera_bracket_link"/>
-    <child link="left_camera_link"/>
-    <origin xyz="0 0 0" rpy="-1.57079632679 0 -1.57079632679"/>
-  </joint>
 </robot>
