Commit message: 关节名修改

File: src/robot_description/urdf/humanoid.gazebo.ros2_control.xacro (robot description, xacro)
@@ -112,4 +112,12 @@
                 <state_interface name="velocity"/>
             </joint>
+            <joint name="left_gripper2_joint">
+                <param name="mimic">left_gripper1_joint</param>
+                <param name="multiplier">-1</param>
+                <command_interface name="position" />
+                <command_interface name="velocity"/>
+                <state_interface name="position" />
+                <state_interface name="velocity"/>
+            </joint>
             <joint name="right_gripper1_joint">
                 <command_interface name="position"/>
@@ -118,4 +126,12 @@
                   <param name="initial_value">${initial_positions['right_gripper1_joint']}</param>
                 </state_interface>
+                <state_interface name="velocity"/>
+            </joint>
+            <joint name="right_gripper2_joint">
+                <param name="mimic">right_gripper1_joint</param>
+                <param name="multiplier">-1</param>
+                <command_interface name="position" />
+                <command_interface name="velocity"/>
+                <state_interface name="position" />
                 <state_interface name="velocity"/>
             </joint>

File: src/robot_description/urdf/humanoid.urdf (robot description, URDF)
Before this commit: robot humanoid, 22 links, 21 joints
Joints:
- removed joint left_gripper2_joiint
- added joint left_gripper2_joint: type prismatic, parent left_wrist_yaw_link, child left_gripper2_link, origin xyz=0 0.14099995082628 -0.0425000000000004 rpy=1.5707963267949 0 -3.14159265358979, axis -1 0 0, limit lower=-0.03 upper=0 effort=20 velocity=50, mimic joint=left_gripper1_joint multiplier=-1.0

Commit message: 解决rqt名称重复bug

File: src/robot_description/urdf/humanoid.gazebo.ros2_control.xacro (robot description, xacro)
@@ -1,5 +1,5 @@
 <?xml version="1.0"?>
 <robot xmlns:xacro="http://www.ros.org/wiki/xacro">
-    <xacro:macro name="humanoid_ros2_control" params="name initial_positions_file">
+    <xacro:macro name="humanoid_gazebo_ros2_control" params="name initial_positions_file">
         <xacro:property name="initial_positions" value="${xacro.load_yaml(initial_positions_file)['initial_positions']}"/>
         <ros2_control name="${name}" type="system">

File: src/robot_description/urdf/humanoid.urdf.xacro (robot description, xacro)
@@ -10,5 +10,5 @@
       <!-- gazebo 仿真 -->
       <xacro:include filename="humanoid.gazebo.ros2_control.xacro" />
-      <xacro:humanoid_ros2_control name="GazeboSystem" initial_positions_file="$(arg initial_positions_file)"/>
+      <xacro:humanoid_gazebo_ros2_control name="GazeboSystem" initial_positions_file="$(arg initial_positions_file)"/>
       <!-- 包含 Gazebo 配置 -->
       <xacro:include filename="humanoid.gazebo.xacro"/>
