Commit message: rearrange the repo

File: RL_training/Isaac_RL/assets/robot_description/urdf/humanoid.urdf (robot description, URDF)
Before this commit: robot humanoid, 22 links, 21 joints
Links:
- link left_gripper2_link: mass 0.0375648373217044 -> 0.0354366119716677
- link right_gripper2_link: mass 0.0375648370970392 -> 0.0393551869062514
Joints:
- joint left_gripper2_joint: origin xyz=0 -0.141 0.0425 rpy=-1.5708 0 3.1416 -> xyz=0 0.14099995082628 -0.0425000000000004 rpy=1.5707963267949 0 -3.14159265358979
- joint right_gripper2_joint: axis -1 0 0 -> 1 0 0; limit lower=0 upper=0.03 effort=20 velocity=50 -> lower=-0.03 upper=0 effort=20 velocity=50; origin xyz=0 0.141 -0.0425 rpy=1.5708 0 3.1416 -> xyz=0 0.141000000000003 -0.0424999999999999 rpy=1.5707963267949 0 3.14159265358979
